File: 12v_connectors.kicad_sch (KiCad schematic)
At the start: 6 parts, among them J4 XT30UPB-F, J5 XT30UPB-F, J6 XT30UPB-F, J7 XT30UPB-F, J8 XT30UPB-F, J9 XT30UPB-F

Commit message: fixed 5 buck aux
Parts:
- J4, J5, J6, J7, J8, J9: footprint XT30UPBF -> power_dist:XT30UPBF
Changed lines of the file:
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@@
 			)
 		)
-		(property "Footprint" "XT30UPBF"
+		(property "Footprint" "power_dist:XT30UPBF"
 			(at 118.11 54.61 0)
 			(hide yes)
@@
 		)
 		(instances
+			(project "24v_power_dist"
+				(path "/351ec213-5341-4e8b-9f3a-42e224a8f757/3b2c23cb-9fa5-4038-939c-e65a02df1393"
+					(reference "J5")
+					(unit 1)
+				)
+			)
 			(project "buck_boost_breakout"
 				(path "/e407faa9-50a3-4231-95da-82dc2233dbf2/3b2c23cb-9fa5-4038-939c-e65a02df1393"
@@
 			)
 		)
-		(property "Footprint" "XT30UPBF"
+		(property "Footprint" "power_dist:XT30UPBF"
 			(at 90.17 54.61 0)
 			(hide yes)
@@
 		)
 		(instances
+			(project "24v_power_dist"
+				(path "/351ec213-5341-4e8b-9f3a-42e224a8f757/3b2c23cb-9fa5-4038-939c-e65a02df1393"
+					(reference "J4")
+					(unit 1)
+				)
+			)
 			(project "buck_boost_breakout"
 				(path "/e407faa9-50a3-4231-95da-82dc2233dbf2/3b2c23cb-9fa5-4038-939c-e65a02df1393"
@@
 			)
 		)
-		(property "Footprint" "XT30UPBF"
+		(property "Footprint" "power_dist:XT30UPBF"
 			(at 203.2 54.61 0)
 			(hide yes)
@@
 		)
 		(instances
+			(project "24v_power_dist"
+				(path "/351ec213-5341-4e8b-9f3a-42e224a8f757/3b2c23cb-9fa5-4038-939c-e65a02df1393"
+					(reference "J8")
+					(unit 1)
+				)
+			)
 			(project "buck_boost_breakout"
 				(path "/e407faa9-50a3-4231-95da-82dc2233dbf2/3b2c23cb-9fa5-4038-939c-e65a02df1393"
@@
 			)
 		)
-		(property "Footprint" "XT30UPBF"
+		(property "Footprint" "power_dist:XT30UPBF"
 			(at 147.32 54.61 0)
 			(hide yes)
@@
 		)
 		(instances
+			(project "24v_power_dist"
+				(path "/351ec213-5341-4e8b-9f3a-42e224a8f757/3b2c23cb-9fa5-4038-939c-e65a02df1393"
+					(reference "J6")
+					(unit 1)
+				)
+			)
 			(project "buck_boost_breakout"
 				(path "/e407faa9-50a3-4231-95da-82dc2233dbf2/3b2c23cb-9fa5-4038-939c-e65a02df1393"
@@
 			)
 		)
-		(property "Footprint" "XT30UPBF"
+		(property "Footprint" "power_dist:XT30UPBF"
 			(at 173.99 54.61 0)
 			(hide yes)
@@
 		)
 		(instances
+			(project "24v_power_dist"
+				(path "/351ec213-5341-4e8b-9f3a-42e224a8f757/3b2c23cb-9fa5-4038-939c-e65a02df1393"
+					(reference "J7")
+					(unit 1)
+				)
+			)
 			(project "buck_boost_breakout"
 				(path "/e407faa9-50a3-4231-95da-82dc2233dbf2/3b2c23cb-9fa5-4038-939c-e65a02df1393"
@@
 			)
 		)
-		(property "Footprint" "XT30UPBF"
+		(property "Footprint" "power_dist:XT30UPBF"
 			(at 232.41 54.61 0)
 			(hide yes)
@@
 		)
 		(instances
+			(project "24v_power_dist"
+				(path "/351ec213-5341-4e8b-9f3a-42e224a8f757/3b2c23cb-9fa5-4038-939c-e65a02df1393"
+					(reference "J9")
+					(unit 1)
+				)
+			)
 			(project "buck_boost_breakout"
 				(path "/e407faa9-50a3-4231-95da-82dc2233dbf2/3b2c23cb-9fa5-4038-939c-e65a02df1393"
@@
 		(dnp no)
 		(fields_autoplaced yes)
-		(property "Reference" "#PWR061"
+		(property "Reference" "#PWR059"
 			(at 58.42 92.71 0)
 			(hide yes)
@@
 		)
 		(instances
+			(project "24v_power_dist"
+				(path "/351ec213-5341-4e8b-9f3a-42e224a8f757/3b2c23cb-9fa5-4038-939c-e65a02df1393"
+					(reference "#PWR059")
+					(unit 1)
+				)
+			)
 			(project "buck_boost_breakout"
 				(path "/e407faa9-50a3-4231-95da-82dc2233dbf2/3b2c23cb-9fa5-4038-939c-e65a02df1393"
