File: 12v_buck.kicad_sch (KiCad schematic)
At the start: 35 parts, among them IC2 LM5116MHX_NOPB

Commit message: fixed 5 buck aux
Parts:
- C54: renamed from C58; footprint (none) -> Capacitor_SMD:C_0603_1608Metric
- C55: renamed from C54; footprint (none) -> Capacitor_SMD:C_0603_1608Metric
- C56: renamed from C53; footprint (none) -> Capacitor_SMD:C_0603_1608Metric
- C58: renamed from C55; footprint (none) -> Capacitor_SMD:C_0603_1608Metric
- C59: renamed from C51; footprint (none) -> Capacitor_SMD:C_0603_1608Metric
- C60: renamed from C50; footprint (none) -> Capacitor_SMD:C_0603_1608Metric
- C61: renamed from C36; footprint (none) -> Capacitor_SMD:C_0603_1608Metric
- C63: renamed from C38; footprint (none) -> Capacitor_SMD:C_0603_1608Metric
- C65: renamed from C44; footprint (none) -> Capacitor_SMD:C_0603_1608Metric
- C66: renamed from C37; footprint (none) -> Capacitor_SMD:C_0603_1608Metric
- C67: renamed from C46; footprint (none) -> Capacitor_SMD:C_0603_1608Metric
- C68: renamed from C39; footprint (none) -> Capacitor_SMD:C_0603_1608Metric
- C69: renamed from C48; footprint (none) -> Capacitor_SMD:C_0603_1608Metric
- C70: renamed from C45; footprint (none) -> Capacitor_SMD:C_0603_1608Metric
- C71: renamed from C47; footprint (none) -> Capacitor_SMD:C_0603_1608Metric
- C72: renamed from C49; footprint (none) -> Capacitor_SMD:C_0603_1608Metric
- R58: renamed from R23; footprint (none) -> power_dist:SVSQ392050R003FTDG
- renumbered C52 to C57, C57 to C62, C56 to C64, D3 to D6, IC2 to IC4, L2 to L4, Q6 to Q10, Q5 to Q9, R29 to R53, R28 to R54, R26 to R55, R27 to R56, R19 to R57, R24 to R59, R25 to R60, R20 to R61, R21 to R62, R22 to R63

Commit message: assigned footprints
Parts:
- C57: footprint (none) -> Capacitor_SMD:C_0603_1608Metric
- C59, C68: footprint Capacitor_SMD:C_0603_1608Metric -> Capacitor_SMD:C_1206_3216Metric
- C61, C66: footprint Capacitor_SMD:C_0603_1608Metric -> power_dist:A786MW157M1JLAS011
- C62, C64: footprint (none) -> power_dist:ESY108M035AL4AA
- R53, R54, R55, R56, R57, R59, R60: footprint (none) -> Resistor_SMD:R_0603_1608Metric
Changed lines of the file:
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@@
 			)
 		)
-		(property "Footprint" ""
+		(property "Footprint" "power_dist:ESY108M035AL4AA"
 			(at 199.39 48.26 0)
 			(hide yes)
@@
 			)
 		)
-		(property "Footprint" ""
+		(property "Footprint" "Resistor_SMD:R_0603_1608Metric"
 			(at 89.662 63.5 90)
 			(hide yes)
@@
 			)
 		)
-		(property "Footprint" ""
+		(property "Footprint" "Resistor_SMD:R_0603_1608Metric"
 			(at 43.942 177.8 90)
 			(hide yes)
@@
 			)
 		)
-		(property "Footprint" ""
+		(property "Footprint" "Resistor_SMD:R_0603_1608Metric"
 			(at 36.83 157.988 90)
 			(hide yes)
@@
 			)
 		)
-		(property "Footprint" "Capacitor_SMD:C_0603_1608Metric"
+		(property "Footprint" "power_dist:A786MW157M1JLAS011"
 			(at 199.39 26.67 0)
 			(hide yes)
@@
 			)
 		)
-		(property "Footprint" "Capacitor_SMD:C_0603_1608Metric"
+		(property "Footprint" "power_dist:A786MW157M1JLAS011"
 			(at 224.79 48.26 0)
 			(hide yes)
@@
 			)
 		)
-		(property "Footprint" "Capacitor_SMD:C_0603_1608Metric"
+		(property "Footprint" "Capacitor_SMD:C_1206_3216Metric"
 			(at 199.39 118.4148 0)
 			(hide yes)
@@
 			)
 		)
-		(property "Footprint" ""
+		(property "Footprint" "power_dist:ESY108M035AL4AA"
 			(at 212.09 48.26 0)
 			(hide yes)
@@
 			)
 		)
-		(property "Footprint" ""
+		(property "Footprint" "Capacitor_SMD:C_0603_1608Metric"
 			(at 121.6152 45.72 0)
 			(hide yes)
@@
 			)
 		)
-		(property "Footprint" "Capacitor_SMD:C_0603_1608Metric"
+		(property "Footprint" "Capacitor_SMD:C_1206_3216Metric"
 			(at 238.4552 52.07 0)
 			(hide yes)
@@
 			)
 		)
-		(property "Footprint" ""
+		(property "Footprint" "Resistor_SMD:R_0603_1608Metric"
 			(at 163.322 34.29 90)
 			(hide yes)
@@
 			)
 		)
-		(property "Footprint" ""
+		(property "Footprint" "Resistor_SMD:R_0603_1608Metric"
 			(at 163.322 48.26 90)
 			(hide yes)
@@
 			)
 		)
-		(property "Footprint" ""
+		(property "Footprint" "Resistor_SMD:R_0603_1608Metric"
 			(at 26.162 50.8 90)
 			(hide yes)
@@
 			)
 		)
-		(property "Footprint" ""
+		(property "Footprint" "Resistor_SMD:R_0603_1608Metric"
 			(at 43.942 163.83 90)
 			(hide yes)
