File: 5v_aux_buck.kicad_sch (KiCad schematic)
At the start: 16 parts, among them IC3 LMR38010SQDDARQ1, J2 Conn_01x02

Commit message: fixed 5 buck aux
Parts:
- removed R34: 0, symbol Device:R
- added R70: 1.5k, Resistor_SMD:R_0603_1608Metric, symbol Device:R
- C2: renamed from C3; footprint (none) -> Capacitor_SMD:C_0603_1608Metric
- C3: renamed from C2; footprint (none) -> Capacitor_SMD:C_0603_1608Metric
- C4: renamed from C1; footprint (none) -> Capacitor_SMD:C_0603_1608Metric
- C5: renamed from C4; footprint (none) -> Capacitor_SMD:C_0603_1608Metric
- L1: renamed from L3; value 27u -> 10u
- R10: renamed from R35; value 6.8k -> 12k; footprint (none) -> Resistor_SMD:R_0603_1608Metric
- R11: renamed from R36; value 430 -> 12k; footprint (none) -> Resistor_SMD:R_0603_1608Metric
- R12: renamed from R37; footprint (none) -> Resistor_SMD:R_0603_1608Metric
- R13: renamed from R38; value 40.2k -> 100k; footprint (none) -> Resistor_SMD:R_0603_1608Metric
- R14: renamed from R39; value 10k -> 24.9k; footprint (none) -> Resistor_SMD:R_0603_1608Metric
- R8: renamed from R40; footprint (none) -> Resistor_SMD:R_0603_1608Metric
- renumbered D4 to D1, IC3 to IC1, J2 to J3
Connections:
- net SYNC: now also R70.2; no longer R10.2
- new net: R10.2, R70.1
Other:
- moved on the sheet: R10, R11

Commit message: assigned footprints
Parts:
- C5: footprint Capacitor_SMD:C_0603_1608Metric -> Capacitor_SMD:C_1206_3216Metric
- J3: footprint (none) -> Connector_PinHeader_2.54mm:PinHeader_1x02_P2.54mm_Vertical
- L1: footprint (none) -> power_dist:IHLP4040DZEE100M01
Changed lines of the file:
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@@
 			)
 		)
-		(property "Footprint" "Capacitor_SMD:C_0603_1608Metric"
+		(property "Footprint" "Capacitor_SMD:C_1206_3216Metric"
 			(at 214.3252 69.85 0)
 			(hide yes)
@@
 			)
 		)
-		(property "Footprint" ""
+		(property "Footprint" "Connector_PinHeader_2.54mm:PinHeader_1x02_P2.54mm_Vertical"
 			(at 69.85 57.15 0)
 			(hide yes)
@@
 			)
 		)
-		(property "Footprint" ""
+		(property "Footprint" "power_dist:IHLP4040DZEE100M01"
 			(at 162.56 59.69 0)
 			(hide yes)
