File: buck_boost.kicad_sch (KiCad schematic)
At the start: 51 parts, among them IC1 LT8705HFE#PBF

Commit message: fixed 5 buck aux
Parts:
- added C77: 4.7u, Capacitor_SMD:C_0603_1608Metric, symbol Device:C
- C10: renamed from C28; footprint (none) -> Capacitor_SMD:C_0603_1608Metric
- C11: renamed from C29; footprint (none) -> Capacitor_SMD:C_0603_1608Metric
- C12: renamed from C24; footprint (none) -> Capacitor_SMD:C_0603_1608Metric
- C13: renamed from C26; footprint (none) -> Capacitor_SMD:C_0603_1608Metric
- C14: renamed from C23; footprint (none) -> Capacitor_SMD:C_0603_1608Metric
- C15: renamed from C27; footprint (none) -> Capacitor_SMD:C_0603_1608Metric
- C16: renamed from C22; footprint (none) -> Capacitor_SMD:C_0603_1608Metric
- C17: renamed from C25; footprint (none) -> Capacitor_SMD:C_0603_1608Metric
- C20: renamed from C41; footprint (none) -> Capacitor_SMD:C_0603_1608Metric
- C22: renamed from C61; footprint (none) -> Capacitor_SMD:C_0603_1608Metric
- C24: renamed from C62; footprint (none) -> Capacitor_SMD:C_0603_1608Metric
- C25: renamed from C43; footprint (none) -> Capacitor_SMD:C_0603_1608Metric
- C26: renamed from C63; footprint (none) -> Capacitor_SMD:C_0603_1608Metric
- C27: renamed from C64; footprint (none) -> Capacitor_SMD:C_0603_1608Metric
- C28: renamed from C65; footprint (none) -> Capacitor_SMD:C_0603_1608Metric
- C29: renamed from C66; footprint (none) -> Capacitor_SMD:C_0603_1608Metric
- C6, C7: footprint (none) -> Capacitor_SMD:C_0603_1608Metric
- C9: renamed from C30; footprint (none) -> Capacitor_SMD:C_0603_1608Metric
- R15: renamed from R1; footprint (none) -> Resistor_SMD:R_0603_1608Metric
- R16: renamed from R30; footprint (none) -> Resistor_SMD:R_0603_1608Metric
- R17: renamed from R2; footprint (none) -> Resistor_SMD:R_0603_1608Metric
- R18: footprint (none) -> Resistor_SMD:R_0603_1608Metric
- R20: renamed from R3; footprint (none) -> Resistor_SMD:R_0603_1608Metric
- R21: renamed from R4; footprint (none) -> Resistor_SMD:R_0603_1608Metric
- R22: renamed from R17; footprint (none) -> Resistor_SMD:R_0603_1608Metric
- R23: renamed from R5; footprint (none) -> Resistor_SMD:R_0603_1608Metric
- R24: renamed from R6; footprint (none) -> Resistor_SMD:R_0603_1608Metric
- R25: renamed from R8; footprint (none) -> Resistor_SMD:R_0603_1608Metric
- renumbered C40 to C18, C59 to C19, C60 to C21, C42 to C23, D1 to D2, D2 to D3, IC1 to IC2, L1 to L2, R13 to R19, R9 to R26, R14 to R27, R7 to R28, R10 to R29, R11 to R30, R12 to R31, R15 to R32, R16 to R33
Connections:
- net GND: now also C77.1
- net at IC2.7 (LDO33), IC2.8 (FBIN): now also C77.2
Other:
- moved on the sheet: R24

Commit message: assigned footprints
Parts:
- added R77, R79: 0, Resistor_SMD:R_0603_1608Metric, symbol Device:R
- C18, C23: footprint (none) -> power_dist:A786MW157M1JLAS011
- C19, C21: footprint (none) -> power_dist:ESY108M035AL4AA
- C20, C25: footprint Capacitor_SMD:C_0603_1608Metric -> Capacitor_SMD:C_1206_3216Metric
- C8: footprint (none) -> Capacitor_SMD:C_0805_2012Metric
- IC2: footprint (none) -> power_dist:LT8705HFEPBF
- R27, R28, R30, R31, R32, R33: footprint (none) -> Resistor_SMD:R_0603_1608Metric
Connections:
- net BATTP: now also R77.1; no longer IC2.37 (CSPIN), R33.1
- net CAPOUT: now also R79.1; no longer IC2.34 (CSPOUT), R32.1
- net CSP: now also R25.1; no longer R25.2
- net at Q2.1 (S), Q2.2 (S), Q2.3 (S)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: now also R25.2; no longer R25.1
- new net CSPIN: IC2.37 (CSPIN), R33.1, R77.2
- new net CSPOUT: IC2.34 (CSPOUT), R32.1, R79.2
Changed lines of the file:
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@@
 	(wire
 		(pts
-			(xy 151.2062 182.9562) (xy 151.2062 151.2062)
+			(xy 245.11 53.34) (xy 256.54 53.34)
 		)
 		(stroke
@@
 	(wire
 		(pts
-			(xy 245.11 53.34) (xy 256.54 53.34)
+			(xy 186.69 104.14) (xy 186.69 115.57)
 		)
 		(stroke
@@
 	(wire
 		(pts
-			(xy 186.69 104.14) (xy 186.69 115.57)
+			(xy 190.5 101.6) (xy 190.5 115.57)
 		)
 		(stroke
@@
 	(wire
 		(pts
+			(xy 66.04 101.6) (xy 66.04 115.57)
+		)
+		(stroke
+			(width 0)
+			(type default)
+		)
+	)
+	(wire
+		(pts
 			(xy 228.6 115.57) (xy 228.6 125.73)
 		)
@@
 	(wire
 		(pts
-			(xy 190.5 104.14) (xy 190.5 115.57)
+			(xy 190.5 83.82) (xy 190.5 93.98)
 		)
 		(stroke
@@
 	(wire
 		(pts
-			(xy 202.0062 182.9562) (xy 151.2062 182.9562)
-		)
-		(stroke
-			(width 0)
-			(type default)
-		)
-	)
-	(wire
-		(pts
 			(xy 232.41 40.64) (xy 232.41 43.18)
 		)
@@
 	(wire
 		(pts
-			(xy 66.04 106.68) (xy 66.04 115.57)
+			(xy 66.04 85.09) (xy 66.04 93.98)
 		)
 		(stroke
@@
 	(wire
 		(pts
-			(xy 237.5662 215.9762) (xy 184.2262 215.9762)
-		)
-		(stroke
-			(width 0)
-			(type default)
-		)
-	)
-	(wire
-		(pts
 			(xy 149.86 148.59) (xy 149.86 154.94)
 		)
@@
 	(wire
 		(pts
-			(xy 202.0062 171.5262) (xy 202.0062 182.9562)
-		)
-		(stroke
-			(width 0)
-			(type default)
-		)
-	)
-	(wire
-		(pts
 			(xy 147.32 137.16) (xy 149.86 137.16)
 		)
@@
 	(wire
 		(pts
-			(xy 184.2262 215.9762) (xy 184.2262 184.2262)
-		)
-		(stroke
-			(width 0)
-			(type default)
-		)
-	)
-	(wire
-		(pts
-			(xy 237.5662 200.7362) (xy 237.5662 215.9762)
-		)
-		(stroke
-			(width 0)
-			(type default)
-		)
-	)
-	(wire
-		(pts
 			(xy 245.11 50.8) (xy 245.11 53.34)
 		)
@@
 	)
 	(label "CSPIN"
-		(at 66.04 106.68 270)
+		(at 66.04 85.09 270)
 		(effects
 			(font
@@
 	)
 	(label "CSPOUT"
-		(at 190.5 104.14 270)
+		(at 190.5 83.82 270)
 		(effects
 			(font
@@
 	)
 	(symbol
+		(lib_id "Device:R")
+		(at 190.5 97.79 180)
+		(unit 1)
+		(body_style 1)
+		(exclude_from_sim no)
+		(in_bom yes)
+		(on_board yes)
+		(in_pos_files yes)
+		(dnp no)
+		(fields_autoplaced yes)
+		(property "Reference" "R79"
+			(at 193.04 96.5199 0)
+			(show_name no)
+			(do_not_autoplace no)
+			(effects
+				(font
+					(size 1.27 1.27)
+				)
+				(justify right)
+			)
+		)
+		(property "Value" "0"
+			(at 193.04 99.0599 0)
+			(show_name no)
+			(do_not_autoplace no)
+			(effects
+				(font
+					(size 1.27 1.27)
+				)
+				(justify right)
+			)
+		)
+		(property "Footprint" "Resistor_SMD:R_0603_1608Metric"
+			(at 192.278 97.79 90)
+			(hide yes)
+			(show_name no)
+			(do_not_autoplace no)
+			(effects
+				(font
+					(size 1.27 1.27)
+				)
+			)
+		)
+		(property "Datasheet" ""
+			(at 190.5 97.79 0)
+			(hide yes)
+			(show_name no)
+			(do_not_autoplace no)
+			(effects
+				(font
+					(size 1.27 1.27)
+				)
+			)
+		)
+		(property "Description" "Resistor"
+			(at 190.5 97.79 0)
+			(hide yes)
+			(show_name no)
+			(do_not_autoplace no)
+			(effects
+				(font
+					(size 1.27 1.27)
+				)
+			)
+		)
+		(pin "1"
+		)
+		(pin "2"
+		)
+		(instances
+			(project "24v_power_dist"
+				(path "/351ec213-5341-4e8b-9f3a-42e224a8f757/0680bbb8-fba3-4e16-8686-501db8d37be5"
+					(reference "R79")
+					(unit 1)
+				)
+				(path "/351ec213-5341-4e8b-9f3a-42e224a8f757/e58c1b29-143d-4dec-a2fb-5e98d5013989"
+					(reference "R80")
+					(unit 1)
+				)
+			)
+		)
+	)
+	(symbol
 		(lib_id "power:GNDPWR")
 		(at 187.96 31.75 0)
@@
 			)
 		)
-		(property "Footprint" "Capacitor_SMD:C_0603_1608Metric"
+		(property "Footprint" "Capacitor_SMD:C_1206_3216Metric"
 			(at 233.3752 50.8 0)
 			(hide yes)
@@
 			)
 		)
-		(property "Footprint" ""
+		(property "Footprint" "power_dist:LT8705HFEPBF"
 			(at 72.39 21.59 0)
 			(hide yes)
@@
 		(lib_id "Device:R")
 		(at 125.73 144.78 0)
-		(mirror y)
+		(mirror x)
 		(unit 1)
 		(body_style 1)
@@
 		(fields_autoplaced yes)
 		(property "Reference" "R25"
-			(at 128.27 143.5099 0)
+			(at 123.19 143.5099 0)
 			(show_name no)
 			(do_not_autoplace no)
@@
 		)
 		(property "Value" "10"
-			(at 128.27 146.0499 0)
+			(at 123.19 146.0499 0)
 			(show_name no)
 			(do_not_autoplace no)
@@
 		)
 		(property "Footprint" "Resistor_SMD:R_0603_1608Metric"
-			(at 127.508 144.78 90)
+			(at 123.952 144.78 90)
 			(hide yes)
 			(show_name no)
@@
 	)
 	(symbol
+		(lib_id "Device:R")
+		(at 66.04 97.79 180)
+		(unit 1)
+		(body_style 1)
+		(exclude_from_sim no)
+		(in_bom yes)
+		(on_board yes)
+		(in_pos_files yes)
+		(dnp no)
+		(fields_autoplaced yes)
+		(property "Reference" "R77"
+			(at 68.58 96.5199 0)
+			(show_name no)
+			(do_not_autoplace no)
+			(effects
+				(font
+					(size 1.27 1.27)
+				)
+				(justify right)
+			)
+		)
+		(property "Value" "0"
+			(at 68.58 99.0599 0)
+			(show_name no)
+			(do_not_autoplace no)
+			(effects
+				(font
+					(size 1.27 1.27)
+				)
+				(justify right)
+			)
+		)
+		(property "Footprint" "Resistor_SMD:R_0603_1608Metric"
+			(at 67.818 97.79 90)
+			(hide yes)
+			(show_name no)
+			(do_not_autoplace no)
+			(effects
+				(font
+					(size 1.27 1.27)
+				)
+			)
+		)
+		(property "Datasheet" ""
+			(at 66.04 97.79 0)
+			(hide yes)
+			(show_name no)
+			(do_not_autoplace no)
+			(effects
+				(font
+					(size 1.27 1.27)
+				)
+			)
+		)
+		(property "Description" "Resistor"
+			(at 66.04 97.79 0)
+			(hide yes)
+			(show_name no)
+			(do_not_autoplace no)
+			(effects
+				(font
+					(size 1.27 1.27)
+				)
+			)
+		)
+		(pin "1"
+		)
+		(pin "2"
+		)
+		(instances
+			(project "24v_power_dist"
+				(path "/351ec213-5341-4e8b-9f3a-42e224a8f757/0680bbb8-fba3-4e16-8686-501db8d37be5"
+					(reference "R77")
+					(unit 1)
+				)
+				(path "/351ec213-5341-4e8b-9f3a-42e224a8f757/e58c1b29-143d-4dec-a2fb-5e98d5013989"
+					(reference "R78")
+					(unit 1)
+				)
+			)
+		)
+	)
+	(symbol
 		(lib_id "Device:C")
 		(at 114.3 101.6 0)
@@
 			)
 		)
-		(property "Footprint" ""
+		(property "Footprint" "power_dist:A786MW157M1JLAS011"
 			(at 219.71 46.99 0)
 			(hide yes)
@@
 			)
 		)
-		(property "Footprint" ""
+		(property "Footprint" "power_dist:ESY108M035AL4AA"
 			(at 194.31 46.99 0)
 			(hide yes)
@@
 			)
 		)
-		(property "Footprint" ""
+		(property "Footprint" "Resistor_SMD:R_0603_1608Metric"
 			(at 255.27 77.978 90)
 			(hide yes)
@@
 			)
 		)
-		(property "Footprint" ""
+		(property "Footprint" "Resistor_SMD:R_0603_1608Metric"
 			(at 226.822 147.32 90)
 			(hide yes)
@@
 			)
 		)
-		(property "Footprint" ""
+		(property "Footprint" "Resistor_SMD:R_0603_1608Metric"
 			(at 226.822 129.54 90)
 			(hide yes)
@@
 			)
 		)
-		(property "Footprint" "Capacitor_SMD:C_0603_1608Metric"
+		(property "Footprint" "Capacitor_SMD:C_1206_3216Metric"
 			(at 207.9752 29.21 0)
 			(hide yes)
@@
 			)
 		)
-		(property "Footprint" ""
+		(property "Footprint" "power_dist:A786MW157M1JLAS011"
 			(at 194.31 25.4 0)
 			(hide yes)
@@
 			)
 		)
-		(property "Footprint" ""
+		(property "Footprint" "Resistor_SMD:R_0603_1608Metric"
 			(at 148.082 144.78 90)
 			(hide yes)
@@
 			)
 		)
-		(property "Footprint" ""
+		(property "Footprint" "Resistor_SMD:R_0603_1608Metric"
 			(at 135.382 64.77 90)
 			(hide yes)
@@
 			)
 		)
-		(property "Footprint" ""
+		(property "Footprint" "power_dist:ESY108M035AL4AA"
 			(at 207.01 46.99 0)
 			(hide yes)
@@
 			)
 		)
-		(property "Footprint" ""
+		(property "Footprint" "Capacitor_SMD:C_0805_2012Metric"
 			(at 52.3748 168.91 0)
 			(hide yes)
@@
 			)
 		)
-		(property "Footprint" ""
+		(property "Footprint" "Resistor_SMD:R_0603_1608Metric"
 			(at 255.27 67.818 90)
 			(hide yes)
