File: ina283aidgkr.kicad_sch (KiCad schematic)
At the start: 3 parts, among them IC5 INA282AIDGKR

Commit message: fixed 5 buck aux
Parts:
- C73: renamed from C5; footprint (none) -> Capacitor_SMD:C_0603_1608Metric
- renumbered R57 to R64
Changed lines of the file:
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@@
 		(dnp no)
 		(fields_autoplaced yes)
-		(property "Reference" "#PWR046"
+		(property "Reference" "#PWR056"
 			(at 147.32 87.63 0)
 			(hide yes)
@@
 		)
 		(instances
+			(project "24v_power_dist"
+				(path "/351ec213-5341-4e8b-9f3a-42e224a8f757/9017cb77-fded-48bc-bce9-ed8cf450d7a7"
+					(reference "#PWR056")
+					(unit 1)
+				)
+			)
 			(project "buck_boost_breakout"
 				(path "/e407faa9-50a3-4231-95da-82dc2233dbf2/9017cb77-fded-48bc-bce9-ed8cf450d7a7"
@@
 		(dnp no)
 		(fields_autoplaced yes)
-		(property "Reference" "#PWR044"
+		(property "Reference" "#PWR057"
 			(at 154.94 110.49 0)
 			(hide yes)
@@
 		)
 		(instances
+			(project "24v_power_dist"
+				(path "/351ec213-5341-4e8b-9f3a-42e224a8f757/9017cb77-fded-48bc-bce9-ed8cf450d7a7"
+					(reference "#PWR057")
+					(unit 1)
+				)
+			)
 			(project "buck_boost_breakout"
 				(path "/e407faa9-50a3-4231-95da-82dc2233dbf2/9017cb77-fded-48bc-bce9-ed8cf450d7a7"
@@
 		(dnp no)
 		(fields_autoplaced yes)
-		(property "Reference" "R57"
+		(property "Reference" "R64"
 			(at 120.65 63.5 0)
 			(show_name no)
@@
 		)
 		(instances
+			(project "24v_power_dist"
+				(path "/351ec213-5341-4e8b-9f3a-42e224a8f757/9017cb77-fded-48bc-bce9-ed8cf450d7a7"
+					(reference "R64")
+					(unit 1)
+				)
+			)
 			(project "buck_boost_breakout"
 				(path "/e407faa9-50a3-4231-95da-82dc2233dbf2/9017cb77-fded-48bc-bce9-ed8cf450d7a7"
@@
 		(dnp no)
 		(fields_autoplaced yes)
-		(property "Reference" "#PWR045"
+		(property "Reference" "#PWR055"
 			(at 90.17 88.9 0)
 			(hide yes)
@@
 		)
 		(instances
+			(project "24v_power_dist"
+				(path "/351ec213-5341-4e8b-9f3a-42e224a8f757/9017cb77-fded-48bc-bce9-ed8cf450d7a7"
+					(reference "#PWR055")
+					(unit 1)
+				)
+			)
 			(project "buck_boost_breakout"
 				(path "/e407faa9-50a3-4231-95da-82dc2233dbf2/9017cb77-fded-48bc-bce9-ed8cf450d7a7"
@@
 		(dnp no)
 		(fields_autoplaced yes)
-		(property "Reference" "C5"
+		(property "Reference" "C73"
 			(at 158.75 95.2499 0)
 			(show_name no)
@@
 			)
 		)
-		(property "Footprint" ""
+		(property "Footprint" "Capacitor_SMD:C_0603_1608Metric"
 			(at 155.9052 100.33 0)
 			(hide yes)
@@
 		)
 		(instances
+			(project "24v_power_dist"
+				(path "/351ec213-5341-4e8b-9f3a-42e224a8f757/9017cb77-fded-48bc-bce9-ed8cf450d7a7"
+					(reference "C73")
+					(unit 1)
+				)
+			)
 			(project "buck_boost_breakout"
 				(path "/e407faa9-50a3-4231-95da-82dc2233dbf2/9017cb77-fded-48bc-bce9-ed8cf450d7a7"
@@
 		)
 		(instances
+			(project "24v_power_dist"
+				(path "/351ec213-5341-4e8b-9f3a-42e224a8f757/9017cb77-fded-48bc-bce9-ed8cf450d7a7"
+					(reference "IC5")
+					(unit 1)
+				)
+			)
 			(project "buck_boost_breakout"
 				(path "/e407faa9-50a3-4231-95da-82dc2233dbf2/9017cb77-fded-48bc-bce9-ed8cf450d7a7"
