File: tempsense.kicad_sch (KiCad schematic)
At the start: 2 parts, among them IC6 TMP1075DGKR

Commit message: fixed 5 buck aux
Parts:
- added C74: .01u, symbol Device:C
- renumbered R58 to R65
Connections:
- net 5V_IN: now also C74.1
- net GND: now also C74.2
Changed lines of the file:
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@@
+	)
+	(junction
+		(at 128.27 104.14)
+		(diameter 0)
+		(color 0 0 0 0)
 	)
 	(junction
@@
 		(color 0 0 0 0)
 	)
+	(junction
+		(at 173.99 96.52)
+		(diameter 0)
+		(color 0 0 0 0)
+	)
+	(wire
+		(pts
+			(xy 173.99 106.68) (xy 173.99 109.22)
+		)
+		(stroke
+			(width 0)
+			(type default)
+		)
+	)
 	(wire
 		(pts
@@
 	(wire
 		(pts
-			(xy 127 104.14) (xy 129.54 104.14)
+			(xy 127 104.14) (xy 128.27 104.14)
 		)
 		(stroke
@@
 	(wire
 		(pts
+			(xy 128.27 104.14) (xy 129.54 104.14)
+		)
+		(stroke
+			(width 0)
+			(type default)
+		)
+	)
+	(wire
+		(pts
 			(xy 157.48 96.52) (xy 166.37 96.52)
 		)
@@
 	(wire
 		(pts
-			(xy 166.37 96.52) (xy 170.18 96.52)
+			(xy 173.99 109.22) (xy 128.27 109.22)
+		)
+		(stroke
+			(width 0)
+			(type default)
+		)
+	)
+	(wire
+		(pts
+			(xy 173.99 96.52) (xy 182.88 96.52)
+		)
+		(stroke
+			(width 0)
+			(type default)
+		)
+	)
+	(wire
+		(pts
+			(xy 166.37 96.52) (xy 173.99 96.52)
+		)
+		(stroke
+			(width 0)
+			(type default)
+		)
+	)
+	(wire
+		(pts
+			(xy 128.27 109.22) (xy 128.27 104.14)
 		)
 		(stroke
@@
 		(pts
 			(xy 166.37 83.82) (xy 114.3 83.82)
+		)
+		(stroke
+			(width 0)
+			(type default)
+		)
+	)
+	(wire
+		(pts
+			(xy 173.99 96.52) (xy 173.99 99.06)
 		)
 		(stroke
@@
 	(hierarchical_label "5V_IN"
 		(shape input)
-		(at 170.18 96.52 0)
+		(at 182.88 96.52 0)
 		(effects
 			(font
@@
 			)
 			(justify right)
+		)
+	)
+	(symbol
+		(lib_id "Device:C")
+		(at 173.99 102.87 0)
+		(unit 1)
+		(body_style 1)
+		(exclude_from_sim no)
+		(in_bom yes)
+		(on_board yes)
+		(in_pos_files yes)
+		(dnp no)
+		(fields_autoplaced yes)
+		(property "Reference" "C74"
+			(at 177.8 101.5999 0)
+			(show_name no)
+			(do_not_autoplace no)
+			(effects
+				(font
+					(size 1.27 1.27)
+				)
+				(justify left)
+			)
+		)
+		(property "Value" ".01u"
+			(at 177.8 104.1399 0)
+			(show_name no)
+			(do_not_autoplace no)
+			(effects
+				(font
+					(size 1.27 1.27)
+				)
+				(justify left)
+			)
+		)
+		(property "Footprint" ""
+			(at 174.9552 106.68 0)
+			(hide yes)
+			(show_name no)
+			(do_not_autoplace no)
+			(effects
+				(font
+					(size 1.27 1.27)
+				)
+			)
+		)
+		(property "Datasheet" ""
+			(at 173.99 102.87 0)
+			(hide yes)
+			(show_name no)
+			(do_not_autoplace no)
+			(effects
+				(font
+					(size 1.27 1.27)
+				)
+			)
+		)
+		(property "Description" "Unpolarized capacitor"
+			(at 173.99 102.87 0)
+			(hide yes)
+			(show_name no)
+			(do_not_autoplace no)
+			(effects
+				(font
+					(size 1.27 1.27)
+				)
+			)
+		)
+		(pin "2"
+		)
+		(pin "1"
+		)
+		(instances
+			(project "24v_power_dist"
+				(path "/351ec213-5341-4e8b-9f3a-42e224a8f757/4009a9ef-11e7-4178-beaa-da09001b5719"
+					(reference "C76")
+					(unit 1)
+				)
+				(path "/351ec213-5341-4e8b-9f3a-42e224a8f757/a8d54f98-7ca4-4f96-a962-1078df78f04b"
+					(reference "C74")
+					(unit 1)
+				)
+				(path "/351ec213-5341-4e8b-9f3a-42e224a8f757/e0d5a034-fc0c-4286-96ba-17430dbde8a3"
+					(reference "C75")
+					(unit 1)
+				)
+			)
 		)
 	)
@@
 		(dnp no)
 		(fields_autoplaced yes)
-		(property "Reference" "R58"
+		(property "Reference" "R65"
 			(at 116.84 91.4399 0)
 			(show_name no)
@@
 		)
 		(instances
+			(project "24v_power_dist"
+				(path "/351ec213-5341-4e8b-9f3a-42e224a8f757/4009a9ef-11e7-4178-beaa-da09001b5719"
+					(reference "R67")
+					(unit 1)
+				)
+				(path "/351ec213-5341-4e8b-9f3a-42e224a8f757/a8d54f98-7ca4-4f96-a962-1078df78f04b"
+					(reference "R65")
+					(unit 1)
+				)
+				(path "/351ec213-5341-4e8b-9f3a-42e224a8f757/e0d5a034-fc0c-4286-96ba-17430dbde8a3"
+					(reference "R66")
+					(unit 1)
+				)
+			)
 			(project "buck_boost_breakout"
 				(path "/e407faa9-50a3-4231-95da-82dc2233dbf2/4009a9ef-11e7-4178-beaa-da09001b5719"
@@
 		)
 		(instances
+			(project "24v_power_dist"
+				(path "/351ec213-5341-4e8b-9f3a-42e224a8f757/4009a9ef-11e7-4178-beaa-da09001b5719"
+					(reference "IC8")
+					(unit 1)
+				)
+				(path "/351ec213-5341-4e8b-9f3a-42e224a8f757/a8d54f98-7ca4-4f96-a962-1078df78f04b"
+					(reference "IC6")
+					(unit 1)
+				)
+				(path "/351ec213-5341-4e8b-9f3a-42e224a8f757/e0d5a034-fc0c-4286-96ba-17430dbde8a3"
+					(reference "IC7")
+					(unit 1)
+				)
+			)
 			(project "buck_boost_breakout"
 				(path "/e407faa9-50a3-4231-95da-82dc2233dbf2/4009a9ef-11e7-4178-beaa-da09001b5719"
@@
 		(dnp no)
 		(fields_autoplaced yes)
-		(property "Reference" "#PWR047"
+		(property "Reference" "#PWR058"
 			(at 120.65 104.14 0)
 			(hide yes)
@@
 		)
 		(instances
+			(project "24v_power_dist"
+				(path "/351ec213-5341-4e8b-9f3a-42e224a8f757/4009a9ef-11e7-4178-beaa-da09001b5719"
+					(reference "#PWR061")
+					(unit 1)
+				)
+				(path "/351ec213-5341-4e8b-9f3a-42e224a8f757/a8d54f98-7ca4-4f96-a962-1078df78f04b"
+					(reference "#PWR058")
+					(unit 1)
+				)
+				(path "/351ec213-5341-4e8b-9f3a-42e224a8f757/e0d5a034-fc0c-4286-96ba-17430dbde8a3"
+					(reference "#PWR060")
+					(unit 1)
+				)
+			)
 			(project "buck_boost_breakout"
 				(path "/e407faa9-50a3-4231-95da-82dc2233dbf2/4009a9ef-11e7-4178-beaa-da09001b5719"

Commit message: assigned footprints
Parts:
- C74: footprint (none) -> Capacitor_SMD:C_0603_1608Metric
- R65: footprint (none) -> Resistor_SMD:R_0603_1608Metric
Connections:
- net 5V_IN: no longer R65.1
- new net 3v3_IN: R65.1
Changed lines of the file:
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@@
 	(paper "A4")
-	(junction
-		(at 166.37 96.52)
-		(diameter 0)
-		(color 0 0 0 0)
-	)
 	(junction
 		(at 128.27 104.14)
@@
 	(wire
 		(pts
-			(xy 166.37 96.52) (xy 166.37 83.82)
-		)
-		(stroke
-			(width 0)
-			(type default)
-		)
-	)
-	(wire
-		(pts
 			(xy 127 104.14) (xy 128.27 104.14)
 		)
@@
 	(wire
 		(pts
-			(xy 157.48 96.52) (xy 166.37 96.52)
-		)
-		(stroke
-			(width 0)
-			(type default)
-		)
-	)
-	(wire
-		(pts
 			(xy 157.48 101.6) (xy 162.56 101.6)
 		)
@@
 	(wire
 		(pts
-			(xy 166.37 96.52) (xy 173.99 96.52)
+			(xy 157.48 96.52) (xy 173.99 96.52)
 		)
 		(stroke
@@
 		(pts
 			(xy 157.48 104.14) (xy 162.56 104.14)
-		)
-		(stroke
-			(width 0)
-			(type default)
-		)
-	)
-	(wire
-		(pts
-			(xy 166.37 83.82) (xy 114.3 83.82)
 		)
 		(stroke
@@
 		(shape output)
 		(at 162.56 101.6 0)
+		(effects
+			(font
+				(size 1.27 1.27)
+			)
+			(justify left)
+		)
+	)
+	(hierarchical_label "3v3_IN"
+		(shape input)
+		(at 114.3 83.82 90)
 		(effects
 			(font
@@
 			)
 		)
-		(property "Footprint" ""
+		(property "Footprint" "Capacitor_SMD:C_0603_1608Metric"
 			(at 174.9552 106.68 0)
 			(hide yes)
@@
 			)
 		)
-		(property "Footprint" ""
+		(property "Footprint" "Resistor_SMD:R_0603_1608Metric"
 			(at 112.522 92.71 90)
 			(hide yes)
